File: board.sch (KiCad schematic (older format))
At the start: 151 parts

Commit message: Generated PCB
Parts:
- C1, C2, C3, C4, C5, C6, C7: renamed from C?; footprint (none) -> Capacitor_SMD:C_0805_2012Metric
- D1, D10, D11, D12, D13, D14, D15, D16, D17, D18, D19, D2, D20, D21, D22, D23, D24, D25, D26, D27, D28, D29, D3, D30, D31, D32, D33, D34, D35, D36, D37, D38, D39, D4, D40, D41, D42, D43, D44, D45, D46, D47, D48, D49, D5, D50, D51, D52, D53, D54, D55, D56, D57, D58, D59, D6, D60, D61, D62, D63, D64, D65, D66, D7, D8, D9: renamed from D?; footprint Diodes_SMD:D_SOD-123 -> Diode_SMD:D_SOD-123
- K_#1, K_#10, K_#2, K_#3, K_#4, K_#5, K_#6, K_#7, K_#8, K_#9: renamed from K_#?; footprint MX_Alps_Hybrid:MX-1U -> MX_Alps_Hybrid:MXOnly-1U-NoLED
- K_'1: renamed from K_'?; footprint MX_Alps_Hybrid:MX-1U -> MX_Alps_Hybrid:MXOnly-1U-NoLED
- K_,1: renamed from K_,?; footprint MX_Alps_Hybrid:MX-1U -> MX_Alps_Hybrid:MXOnly-1U-NoLED
- K_-1: renamed from K_-?; footprint MX_Alps_Hybrid:MX-1U -> MX_Alps_Hybrid:MXOnly-1U-NoLED
- K_.1: renamed from K_.?; footprint MX_Alps_Hybrid:MX-1U -> MX_Alps_Hybrid:MXOnly-1U-NoLED
- K_/1: renamed from K_/?; footprint MX_Alps_Hybrid:MX-1U -> MX_Alps_Hybrid:MXOnly-1U-NoLED
- K_;1: renamed from K_;?; footprint MX_Alps_Hybrid:MX-1U -> MX_Alps_Hybrid:MXOnly-1U-NoLED
- K_=1: renamed from K_=?; footprint MX_Alps_Hybrid:MX-1U -> MX_Alps_Hybrid:MXOnly-1U-NoLED
- K_A1: renamed from K_A?; footprint MX_Alps_Hybrid:MX-1U -> MX_Alps_Hybrid:MXOnly-1U-NoLED
- K_ALT1: renamed from K_ALT?; footprint MX_Alps_Hybrid:MX-1.25U -> MX_Alps_Hybrid:MXOnly-1.25U-NoLED
- K_B1: renamed from K_B?; footprint MX_Alps_Hybrid:MX-1U -> MX_Alps_Hybrid:MXOnly-1U-NoLED
- K_BACK1: renamed from K_BACK?; footprint MX_Alps_Hybrid:MX-2U -> MX_Alps_Hybrid:MXOnly-2U-NoLED
- K_C1: renamed from K_C?; footprint MX_Alps_Hybrid:MX-1U -> MX_Alps_Hybrid:MXOnly-1U-NoLED
- K_CAPS1: renamed from K_CAPS?; footprint MX_Alps_Hybrid:MX-1.75U -> MX_Alps_Hybrid:MXOnly-1.75U-NoLED
- K_CTRL1: renamed from K_CTRL?; footprint MX_Alps_Hybrid:MX-1.25U -> MX_Alps_Hybrid:MXOnly-1.25U-NoLED
- K_D1: renamed from K_D?; footprint MX_Alps_Hybrid:MX-1U -> MX_Alps_Hybrid:MXOnly-1U-NoLED
- K_DELETE1: renamed from K_DELETE?; footprint MX_Alps_Hybrid:MX-2U -> MX_Alps_Hybrid:MXOnly-2U-NoLED
- K_DOWN1: renamed from K_DOWN?; footprint MX_Alps_Hybrid:MX-1U -> MX_Alps_Hybrid:MXOnly-1U-NoLED
- K_E1: renamed from K_E?; footprint MX_Alps_Hybrid:MX-1U -> MX_Alps_Hybrid:MXOnly-1U-NoLED
- K_ENTER1: renamed from K_ENTER?; footprint MX_Alps_Hybrid:MX-2.25U -> MX_Alps_Hybrid:MXOnly-2.25U-NoLED
- K_ESC1: renamed from K_ESC?; footprint MX_Alps_Hybrid:MX-1U -> MX_Alps_Hybrid:MXOnly-1U-NoLED
- K_F1: renamed from K_F?; footprint MX_Alps_Hybrid:MX-1U -> MX_Alps_Hybrid:MXOnly-1U-NoLED
- K_G1: renamed from K_G?; footprint MX_Alps_Hybrid:MX-1U -> MX_Alps_Hybrid:MXOnly-1U-NoLED
- K_H1: renamed from K_H?; footprint MX_Alps_Hybrid:MX-1U -> MX_Alps_Hybrid:MXOnly-1U-NoLED
- K_I1: renamed from K_I?; footprint MX_Alps_Hybrid:MX-1U -> MX_Alps_Hybrid:MXOnly-1U-NoLED
- K_INSERT1: renamed from K_INSERT?; footprint MX_Alps_Hybrid:MX-2U -> MX_Alps_Hybrid:MXOnly-2U-NoLED
- K_J1: renamed from K_J?; footprint MX_Alps_Hybrid:MX-1U -> MX_Alps_Hybrid:MXOnly-1U-NoLED
- K_K1: renamed from K_K?; footprint MX_Alps_Hybrid:MX-1U -> MX_Alps_Hybrid:MXOnly-1U-NoLED
- K_L1: renamed from K_L?; footprint MX_Alps_Hybrid:MX-1U -> MX_Alps_Hybrid:MXOnly-1U-NoLED
- K_LEFT1: renamed from K_LEFT?; footprint MX_Alps_Hybrid:MX-1U -> MX_Alps_Hybrid:MXOnly-1U-NoLED
- K_M1: renamed from K_M?; footprint MX_Alps_Hybrid:MX-1U -> MX_Alps_Hybrid:MXOnly-1U-NoLED
- K_N1: renamed from K_N?; footprint MX_Alps_Hybrid:MX-1U -> MX_Alps_Hybrid:MXOnly-1U-NoLED
- K_O1: renamed from K_O?; footprint MX_Alps_Hybrid:MX-1U -> MX_Alps_Hybrid:MXOnly-1U-NoLED
- K_P1: renamed from K_P?; footprint MX_Alps_Hybrid:MX-1U -> MX_Alps_Hybrid:MXOnly-1U-NoLED
- K_Q1: renamed from K_Q?; footprint MX_Alps_Hybrid:MX-1U -> MX_Alps_Hybrid:MXOnly-1U-NoLED
- K_R1: renamed from K_R?; footprint MX_Alps_Hybrid:MX-1U -> MX_Alps_Hybrid:MXOnly-1U-NoLED
- K_RALT1: renamed from K_RALT?; footprint MX_Alps_Hybrid:MX-1.25U-FLIPPED -> MX_Alps_Hybrid:MXOnly-1.25U-NoLED
- K_RCTRL1: renamed from K_RCTRL?; footprint MX_Alps_Hybrid:MX-1.25U -> MX_Alps_Hybrid:MXOnly-1.25U-NoLED
- K_RFN1: renamed from K_RFN?; footprint MX_Alps_Hybrid:MX-1.25U -> MX_Alps_Hybrid:MXOnly-1.25U-NoLED
- K_RIGHT1: renamed from K_RIGHT?; footprint MX_Alps_Hybrid:MX-1U -> MX_Alps_Hybrid:MXOnly-1U-NoLED
- K_RSHIFT1: renamed from K_RSHIFT?; footprint MX_Alps_Hybrid:MX-2.75U-FLIPPED -> MX_Alps_Hybrid:MXOnly-2.75U-NoLED
- K_S1: renamed from K_S?; footprint MX_Alps_Hybrid:MX-1U -> MX_Alps_Hybrid:MXOnly-1U-NoLED
- K_SHIFT1: renamed from K_SHIFT?; footprint MX_Alps_Hybrid:MX-2.25U -> MX_Alps_Hybrid:MXOnly-2.25U-NoLED
- K_SPACE1: renamed from K_SPACE?; footprint MX_Alps_Hybrid:MX-6.25U-ReversedStabilizers -> MX_Alps_Hybrid:MXOnly-6.25U-NoLED
- K_T1: renamed from K_T?; footprint MX_Alps_Hybrid:MX-1U -> MX_Alps_Hybrid:MXOnly-1U-NoLED
- K_TAB1: renamed from K_TAB?; footprint MX_Alps_Hybrid:MX-1.5U -> MX_Alps_Hybrid:MXOnly-1.5U-NoLED
- K_U1: renamed from K_U?; footprint MX_Alps_Hybrid:MX-1U -> MX_Alps_Hybrid:MXOnly-1U-NoLED
- K_UP1: renamed from K_UP?; footprint MX_Alps_Hybrid:MX-1U -> MX_Alps_Hybrid:MXOnly-1U-NoLED
- K_V1: renamed from K_V?; footprint MX_Alps_Hybrid:MX-1U -> MX_Alps_Hybrid:MXOnly-1U-NoLED
- K_W1: renamed from K_W?; footprint MX_Alps_Hybrid:MX-1U -> MX_Alps_Hybrid:MXOnly-1U-NoLED
- K_WIN1: renamed from K_WIN?; footprint MX_Alps_Hybrid:MX-1U-FLIPPED -> MX_Alps_Hybrid:MXOnly-1U-NoLED
- K_X1: renamed from K_X?; footprint MX_Alps_Hybrid:MX-1U -> MX_Alps_Hybrid:MXOnly-1U-NoLED
- K_Y1: renamed from K_Y?; footprint MX_Alps_Hybrid:MX-1U -> MX_Alps_Hybrid:MXOnly-1U-NoLED
- K_Z1: renamed from K_Z?; footprint MX_Alps_Hybrid:MX-1U -> MX_Alps_Hybrid:MXOnly-1U-NoLED
- K_[1: renamed from K_[?; footprint MX_Alps_Hybrid:MX-1U -> MX_Alps_Hybrid:MXOnly-1U-NoLED
- K_\1: renamed from K_\?; footprint MX_Alps_Hybrid:MX-1.5U -> MX_Alps_Hybrid:MXOnly-1U-NoLED
- K_]1: renamed from K_]?; footprint MX_Alps_Hybrid:MX-1U -> MX_Alps_Hybrid:MXOnly-1U-NoLED
- R1, R2: renamed from R?; footprint (none) -> Resistor_SMD:R_0805_2012Metric
- R3, R4, R5, R6: renamed from R?; footprint Resistors_SMD:R_0805 -> Resistor_SMD:R_0805_2012Metric
- SW1: renamed from SW?; footprint (none) -> random-keyboard-parts:Molex-0548190589
- Y1: renamed from Y?; footprint (none) -> Crystal:Crystal_SMD_3225-4Pin_3.2x2.5mm
- gave numbers to parts that had none: 4

Commit message: PCB layout first pass
Parts:
- K_DELETE1, K_INSERT1: value MX-2U -> MX-1U; footprint MX_Alps_Hybrid:MXOnly-2U-NoLED -> MX_Alps_Hybrid:MXOnly-1U-NoLED
- K_RSHIFT1: value MX-2.75U -> MX-2.25U; footprint MX_Alps_Hybrid:MXOnly-2.75U-NoLED -> MX_Alps_Hybrid:MXOnly-2.25U-NoLED
- K_\1: footprint MX_Alps_Hybrid:MXOnly-1U-NoLED -> MX_Alps_Hybrid:MXOnly-1.5U-NoLED; symbol MX_Alps_Hybrids:MX-1U -> MX_Alps_Hybrids:MX-1.5U
Changed lines of the file:
@@
 $EndComp
 $Comp
-L MX_Alps_Hybrids:MX-1U K_\1
+L MX_Alps_Hybrids:MX-1.5U K_\1
 U 1 1 5C993BCD
 P 13200 2850
 F 0 "K_\\1" H 13200 2975 60  0000 C CNN
 F 1 "MX-1.5U" H 13200 2900 20  0000 C CNN
-F 2 "MX_Alps_Hybrid:MXOnly-1U-NoLED" H 13175 2825 60  0001 C CNN
+F 2 "MX_Alps_Hybrid:MXOnly-1.5U-NoLED" H 13175 2825 60  0001 C CNN
 F 3 "" H 13175 2825 60  0001 C CNN
 	1    13200 2850
@@
 P 12600 4150
 F 0 "K_RSHIFT1" H 12600 4275 60  0000 C CNN
-F 1 "MX-2.75U" H 12600 4200 20  0000 C CNN
-F 2 "MX_Alps_Hybrid:MXOnly-2.75U-NoLED" H 12575 4125 60  0001 C CNN
+F 1 "MX-2.25U" H 12600 4200 20  0000 C CNN
+F 2 "MX_Alps_Hybrid:MXOnly-2.25U-NoLED" H 12575 4125 60  0001 C CNN
 F 3 "" H 12575 4125 60  0001 C CNN
 	1    12600 4150
@@
 P 14400 2200
 F 0 "K_INSERT1" H 14400 2325 60  0000 C CNN
-F 1 "MX-2U" H 14400 2250 20  0000 C CNN
-F 2 "MX_Alps_Hybrid:MXOnly-2U-NoLED" H 14375 2175 60  0001 C CNN
+F 1 "MX-1U" H 14400 2250 20  0000 C CNN
+F 2 "MX_Alps_Hybrid:MXOnly-1U-NoLED" H 14375 2175 60  0001 C CNN
 F 3 "" H 14375 2175 60  0001 C CNN
 	1    14400 2200
@@
 P 14400 2850
 F 0 "K_DELETE1" H 14400 2975 60  0000 C CNN
-F 1 "MX-2U" H 14400 2900 20  0000 C CNN
-F 2 "MX_Alps_Hybrid:MXOnly-2U-NoLED" H 14375 2825 60  0001 C CNN
+F 1 "MX-1U" H 14400 2900 20  0000 C CNN
+F 2 "MX_Alps_Hybrid:MXOnly-1U-NoLED" H 14375 2825 60  0001 C CNN
 F 3 "" H 14375 2825 60  0001 C CNN
 	1    14400 2850

Commit message: Fixes
Parts:
- SW1: footprint random-keyboard-parts:Molex-0548190589 -> random-keyboard-parts:PushButton_6x6mm_TH_Pretty
- renumbered K_RFN1 to K_FN1
Changed lines of the file:
@@
 F 0 "SW1" H 1800 1835 50  0000 C CNN
 F 1 "5.2x5.2mm" H 1800 1744 50  0000 C CNN
-F 2 "random-keyboard-parts:Molex-0548190589" H 1800 1750 50  0001 C CNN
+F 2 "random-keyboard-parts:PushButton_6x6mm_TH_Pretty" H 1800 1750 50  0001 C CNN
 F 3 "" H 1800 1750 50  0001 C CNN
 	1    1800 1550
@@
 $EndComp
 $Comp
-L MX_Alps_Hybrids:MX-1U K_RFN1
+L MX_Alps_Hybrids:MX-1U K_FN1
 U 1 1 5C994176
 P 12000 4800
-F 0 "K_RFN1" H 12000 4925 60  0000 C CNN
+F 0 "K_FN1" H 12000 4925 60  0000 C CNN
 F 1 "MX-1.25U" H 12000 4850 20  0000 C CNN
 F 2 "MX_Alps_Hybrid:MXOnly-1.25U-NoLED" H 11975 4775 60  0001 C CNN

Commit message: More fixes
Parts:
- SW1: footprint random-keyboard-parts:PushButton_6x6mm_TH_Pretty -> random-keyboard-parts:PushButton_6x6mm_TH
Changed lines of the file:
@@
 F 0 "SW1" H 1800 1835 50  0000 C CNN
 F 1 "5.2x5.2mm" H 1800 1744 50  0000 C CNN
-F 2 "random-keyboard-parts:PushButton_6x6mm_TH_Pretty" H 1800 1750 50  0001 C CNN
+F 2 "random-keyboard-parts:PushButton_6x6mm_TH" H 1800 1750 50  0001 C CNN
 F 3 "" H 1800 1750 50  0001 C CNN
 	1    1800 1550

Commit message: Route around USB, missing fuse
Parts:
- F1: footprint Fuse_Holders_and_Fuses:Fuse_SMD1206_Reflow -> Fuse:Fuse_1206_3216Metric
Changed lines of the file:
@@
 F 0 "F1" V 2475 5850 50  0000 C CNN
 F 1 "500mA" V 2625 5850 50  0000 C CNN
-F 2 "Fuse_Holders_and_Fuses:Fuse_SMD1206_Reflow" H 2600 5650 50  0001 L CNN
+F 2 "Fuse:Fuse_1206_3216Metric" H 2600 5650 50  0001 L CNN
 F 3 "" H 2550 5850 50  0001 C CNN
 	1    2550 5850
