File: board_arm.sch (KiCad schematic (older format))
At the start: 150 parts, among them SW2 SW_Push, U2 PRTR5V0U2X, U3 STM32F072CBT6

Commit message: ARM board
Parts:
- added C5, C6: 4.7uF, Capacitor_SMD:C_0805_2012Metric, symbol Device:C_Small
- added C7: 10nF, Capacitor_SMD:C_0805_2012Metric, symbol Device:C_Small
- added C8: 1uF, Capacitor_SMD:C_0805_2012Metric, symbol Device:C_Small
- C10, C11, C9: renamed from C?; footprint (none) -> Capacitor_SMD:C_0805_2012Metric
- C4: renamed from C7; value 10uF -> 0.1uF
- R1: renamed from R2; footprint Resistors_SMD:R_0805 -> Resistor_SMD:R_0805_2012Metric
- R2, R3: renamed from R?; footprint Resistors_SMD:R_0805 -> Resistor_SMD:R_0805_2012Metric
- U3: renamed from U?; footprint SOIC127P600X175-8N -> locallib:MCP1725-3302E_SN
- gave numbers to parts that had none: 1
- renumbered C4 to C1, C5 to C2, C6 to C3, R5 to R4, R6 to R5, SW2 to SW1, U3 to U1
Connections:
- net labels added: SWDCLK, SWDIO
- wire segments 297 -> 309
Other:
- moved on the sheet: C1, C10, C11, C2, C3, C4, C9, R1, R2, R3, SW2, U1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

Commit message: Fix MCU wires
Parts:
- U1: footprint Package_QFP:LQFP-32_7x7mm_P0.8mm -> Package_QFP:LQFP-48_7x7mm_P0.5mm
Changed lines of the file:
@@
 Wire Wire Line
 	1525 5500 1525 5400
-Connection ~ 1525 5400
 Wire Wire Line
 	1525 5200 1525 5100
-Connection ~ 1525 5200
 Connection ~ 1675 5400
-Wire Wire Line
-	1525 5400 1675 5400
 Wire Wire Line
 	1975 5400 1675 5400
 Connection ~ 1675 5200
-Wire Wire Line
-	1675 5200 1975 5200
-Wire Wire Line
-	1675 5200 1525 5200
 Connection ~ 1375 5400
-Wire Wire Line
-	1375 5400 1525 5400
 Wire Wire Line
 	1075 5400 1375 5400
 Connection ~ 1375 5200
-Wire Wire Line
-	1525 5200 1375 5200
 Wire Wire Line
 	1375 5200 1075 5200
@@
 	1    0    0    -1
 $EndComp
-Text GLabel 4050 6575 2    60   Input ~ 0
-D-
-Text GLabel 4050 6675 2    60   Input ~ 0
-D+
 $Comp
 L Type-C:HRO-TYPE-C-31-M-12 USB?
@@
 F 0 "U1" H 3075 1439 50  0000 C CNN
 F 1 "STM32F072CBT6" H 3075 1348 50  0000 C CNN
-F 2 "Package_QFP:LQFP-32_7x7mm_P0.8mm" H 2725 2125 50  0001 R CNN
+F 2 "Package_QFP:LQFP-48_7x7mm_P0.5mm" H 2725 2125 50  0001 R CNN
 F 3 "http://www.st.com/st-web-ui/static/active/en/resource/technical/document/datasheet/DM00105814.pdf" H 3125 3025 50  0001 C CNN
 	1    3125 3025
 	1    0    0    -1
 $EndComp
-Text GLabel 3725 4025 2    50   Input ~ 0
-D+
-Text GLabel 3725 3925 2    50   Input ~ 0
-D-
 Wire Wire Line
 	2575 6675 4050 6675
@@
 Wire Wire Line
 	2800 5400 3075 5400
+Wire Wire Line
+	1375 5400 1525 5400
+Wire Wire Line
+	1525 5400 1675 5400
+Connection ~ 1525 5400
+Wire Wire Line
+	1675 5200 1975 5200
+Wire Wire Line
+	1525 5200 1375 5200
+Wire Wire Line
+	1675 5200 1525 5200
+Connection ~ 1525 5200
+Text GLabel 4050 6575 2    50   Input ~ 0
+D-
+Text GLabel 3725 3925 2    50   Input ~ 0
+D-
+Text GLabel 4050 6675 2    50   Input ~ 0
+D+
+Text GLabel 3725 4025 2    50   Input ~ 0
+D+
 $EndSCHEMATC

Commit message: Pretty
Connections:
- wire segments 309 -> 318
Changed lines of the file:
@@
 AR Path="/5C82C6C8/5C8D49F2" Ref="R?"  Part="1"
 AR Path="/5C8D49F2" Ref="R4"  Part="1"
-F 0 "R4" H 2505 7345 50  0000 L CNN
-F 1 "5.1k" H 2505 7285 50  0000 L CNN
+F 0 "R4" V 2550 7325 50  0000 C CNN
+F 1 "5.1k" V 2625 7325 50  0000 C CNN
 F 2 "Resistor_SMD:R_0805_2012Metric" H 2475 7325 50  0001 C CNN
 F 3 "" H 2475 7325 50  0001 C CNN
@@
 AR Path="/5C82C6C8/5C8D49F9" Ref="R?"  Part="1"
 AR Path="/5C8D49F9" Ref="R5"  Part="1"
-F 0 "R5" H 2505 7595 50  0000 L CNN
-F 1 "5.1k" H 2505 7535 50  0000 L CNN
+F 0 "R5" V 2550 7575 50  0000 C CNN
+F 1 "5.1k" V 2625 7575 50  0000 C CNN
 F 2 "Resistor_SMD:R_0805_2012Metric" H 2475 7575 50  0001 C CNN
 F 3 "" H 2475 7575 50  0001 C CNN
@@
 AR Path="/5C82C6C8/5C8D4A28" Ref="U?"  Part="1"
 AR Path="/5C8D4A28" Ref="U2"  Part="1"
-F 0 "U2" H 3025 7347 60  0000 C CNN
-F 1 "PRTR5V0U2X" H 3025 7241 60  0000 C CNN
+F 0 "U2" H 3025 7325 60  0000 C CNN
+F 1 "PRTR5V0U2X" H 3025 7225 60  0000 C CNN
 F 2 "locallib:SOT143B" H 3025 7050 60  0001 C CNN
 F 3 "" H 3025 7050 60  0001 C CNN
@@
 AR Path="/5C8D4A31" Ref="#PWR0115"  Part="1"
 F 0 "#PWR0115" H 3425 6850 50  0001 C CNN
-F 1 "VCC" H 3442 7173 50  0000 C CNN
+F 1 "VCC" H 3425 7175 50  0000 C CNN
 F 2 "" H 3425 7000 50  0001 C CNN
 F 3 "" H 3425 7000 50  0001 C CNN
@@
 AR Path="/5C7BFB71" Ref="#PWR0120"  Part="1"
 F 0 "#PWR0120" H 1625 1225 50  0001 C CNN
-F 1 "GND" H 1630 1302 50  0000 C CNN
+F 1 "GND" H 1625 1325 50  0000 C CNN
 F 2 "" H 1625 1475 50  0001 C CNN
 F 3 "" H 1625 1475 50  0001 C CNN
@@
 L power:GND #PWR0101
 U 1 1 5C7DAA6D
-P 2650 4650
-F 0 "#PWR0101" H 2650 4400 50  0001 C CNN
-F 1 "GND" H 2655 4477 50  0000 C CNN
-F 2 "" H 2650 4650 50  0001 C CNN
-F 3 "" H 2650 4650 50  0001 C CNN
-	1    2650 4650
+P 2600 4600
+F 0 "#PWR0101" H 2600 4350 50  0001 C CNN
+F 1 "GND" H 2605 4427 50  0000 C CNN
+F 2 "" H 2600 4600 50  0001 C CNN
+F 3 "" H 2600 4600 50  0001 C CNN
+	1    2600 4600
 	1    0    0    -1
 $EndComp
@@
 AR Path="/5C70FC4F/5C83E985" Ref="SW?"  Part="1"
 AR Path="/5C83E985" Ref="SW2"  Part="1"
-F 0 "SW2" H 1300 1600 50  0000 C CNN
-F 1 "SW_SPDT" H 1300 1691 50  0000 C CNN
+F 0 "SW2" H 1300 1625 50  0000 C CNN
+F 1 "SW_SPDT" H 1300 1725 50  0000 C CNN
 F 2 "Button_Switch_SMD:SW_SPDT_PCM12" H 1300 1925 50  0001 C CNN
 F 3 "" H 1300 1925 50  0001 C CNN
@@
 AR Path="/5C70FC4F/5C83E98C" Ref="R?"  Part="1"
 AR Path="/5C83E98C" Ref="R1"  Part="1"
-F 0 "R1" V 1529 1925 50  0000 C CNN
-F 1 "10k" V 1620 1925 50  0000 C CNN
+F 0 "R1" V 1800 1925 50  0000 C CNN
+F 1 "10k" V 1875 1925 50  0000 C CNN
 F 2 "Resistor_SMD:R_0805_2012Metric" H 1725 1925 50  0001 C CNN
 F 3 "~" H 1725 1925 50  0001 C CNN
@@
 AR Path="/5C83E99B" Ref="#PWR0103"  Part="1"
 F 0 "#PWR0103" H 975 1675 50  0001 C CNN
-F 1 "+3V3" H 990 1998 50  0000 C CNN
+F 1 "+3V3" H 975 2000 50  0000 C CNN
 F 2 "" H 975 1825 50  0001 C CNN
 F 3 "" H 975 1825 50  0001 C CNN
@@
 AR Path="/5C70FC4F/5C9A09D2" Ref="R?"  Part="1"
 AR Path="/5C9A09D2" Ref="R3"  Part="1"
-F 0 "R3" V 7129 6800 50  0000 C CNN
-F 1 "10k" V 7220 6800 50  0000 C CNN
+F 0 "R3" H 7275 6750 50  0000 R CNN
+F 1 "10k" H 7275 6850 50  0000 R CNN
 F 2 "Resistor_SMD:R_0805_2012Metric" H 7325 6800 50  0001 C CNN
 F 3 "~" H 7325 6800 50  0001 C CNN
@@
 P 5150 6525
 F 0 "#PWR0109" H 5150 6375 50  0001 C CNN
-F 1 "+5V" H 5165 6698 50  0000 C CNN
+F 1 "+5V" H 5150 6700 50  0000 C CNN
 F 2 "" H 5150 6525 50  0001 C CNN
 F 3 "" H 5150 6525 50  0001 C CNN
@@
 AR Path="/5C70FC4F/5CED8667" Ref="R?"  Part="1"
 AR Path="/5CED8667" Ref="R2"  Part="1"
-F 0 "R2" V 5029 6750 50  0000 C CNN
-F 1 "10k" V 5120 6750 50  0000 C CNN
+F 0 "R2" H 5150 6800 50  0000 R CNN
+F 1 "10k" H 5150 6700 50  0000 R CNN
 F 2 "Resistor_SMD:R_0805_2012Metric" H 5225 6750 50  0001 C CNN
 F 3 "~" H 5225 6750 50  0001 C CNN
@@
 Wire Wire Line
 	5425 6600 5650 6600
-Connection ~ 3125 1525
-Wire Wire Line
-	3125 1525 3225 1525
-Connection ~ 3225 1525
-Wire Wire Line
-	3225 1525 3325 1525
-Connection ~ 3325 1525
-Wire Wire Line
-	2925 1525 3025 1525
-Connection ~ 3025 1525
-Wire Wire Line
-	3025 1525 3125 1525
-Connection ~ 2925 4525
-Wire Wire Line
-	2925 4525 3025 4525
-Connection ~ 3025 4525
-Wire Wire Line
-	3025 4525 3125 4525
-Connection ~ 3125 4525
-Wire Wire Line
-	3125 4525 3225 4525
-Wire Wire Line
-	2650 4525 2650 4650
-Wire Wire Line
-	2650 4525 2925 4525
-Wire Wire Line
-	3500 1525 3500 1400
-Wire Wire Line
-	3325 1525 3500 1525
 Wire Wire Line
 	1825 1925 2425 1925
@@
 Text GLabel 3725 4025 2    50   Input ~ 0
 D+
+Wire Wire Line
+	3225 4525 3225 4550
+Wire Wire Line
+	3225 4550 3125 4550
+Wire Wire Line
+	2600 4550 2600 4600
+Wire Wire Line
+	2925 4525 2925 4550
+Connection ~ 2925 4550
+Wire Wire Line
+	2925 4550 2600 4550
+Wire Wire Line
+	3025 4525 3025 4550
+Connection ~ 3025 4550
+Wire Wire Line
+	3025 4550 2925 4550
+Wire Wire Line
+	3125 4525 3125 4550
+Connection ~ 3125 4550
+Wire Wire Line
+	3125 4550 3025 4550
+Wire Wire Line
+	2925 1525 2925 1500
+Wire Wire Line
+	2925 1500 3025 1500
+Wire Wire Line
+	3500 1500 3500 1400
+Wire Wire Line
+	3025 1525 3025 1500
+Connection ~ 3025 1500
+Wire Wire Line
+	3025 1500 3125 1500
+Wire Wire Line
+	3125 1525 3125 1500
+Connection ~ 3125 1500
+Wire Wire Line
+	3125 1500 3225 1500
+Wire Wire Line
+	3225 1525 3225 1500
+Connection ~ 3225 1500
+Wire Wire Line
+	3225 1500 3325 1500
+Wire Wire Line
+	3325 1525 3325 1500
+Connection ~ 3325 1500
+Wire Wire Line
+	3325 1500 3500 1500
 $EndSCHEMATC

Commit message: More fixes
Parts:
- removed SW1: SW_Push, Button_Switch_SMD:SW_SPST_SKQG_WithoutStem, symbol Switch:SW_Push
- SW1: renamed from SW2; footprint Button_Switch_SMD:SW_SPDT_PCM12 -> locallib:SW_SPDT_9.0x3.5mm
Connections:
- wire segments 318 -> 314
Other:
- moved on the sheet: C1, C2, C3, C4, C5, C6, C7, C8
Changed lines of the file:
@@
 L Device:C_Small C1
 U 1 1 5C603E42
-P 1075 5300
-F 0 "C1" H 1167 5346 50  0000 L CNN
-F 1 "0.1uF" H 1167 5255 50  0000 L CNN
-F 2 "Capacitor_SMD:C_0805_2012Metric" H 1075 5300 50  0001 C CNN
-F 3 "~" H 1075 5300 50  0001 C CNN
-	1    1075 5300
+P 1075 5275
+F 0 "C1" H 1167 5321 50  0000 L CNN
+F 1 "0.1uF" H 1167 5230 50  0000 L CNN
+F 2 "Capacitor_SMD:C_0805_2012Metric" H 1075 5275 50  0001 C CNN
+F 3 "~" H 1075 5275 50  0001 C CNN
+	1    1075 5275
 	1    0    0    -1
 $EndComp
@@
 L Device:C_Small C2
 U 1 1 5C603F7E
-P 1375 5300
-F 0 "C2" H 1467 5346 50  0000 L CNN
-F 1 "0.1uF" H 1467 5255 50  0000 L CNN
-F 2 "Capacitor_SMD:C_0805_2012Metric" H 1375 5300 50  0001 C CNN
-F 3 "~" H 1375 5300 50  0001 C CNN
-	1    1375 5300
+P 1450 5275
+F 0 "C2" H 1542 5321 50  0000 L CNN
+F 1 "0.1uF" H 1542 5230 50  0000 L CNN
+F 2 "Capacitor_SMD:C_0805_2012Metric" H 1450 5275 50  0001 C CNN
+F 3 "~" H 1450 5275 50  0001 C CNN
+	1    1450 5275
 	1    0    0    -1
 $EndComp
@@
 L Device:C_Small C3
 U 1 1 5C603FAE
-P 1675 5300
-F 0 "C3" H 1767 5346 50  0000 L CNN
-F 1 "0.1uF" H 1767 5255 50  0000 L CNN
-F 2 "Capacitor_SMD:C_0805_2012Metric" H 1675 5300 50  0001 C CNN
-F 3 "~" H 1675 5300 50  0001 C CNN
-	1    1675 5300
+P 1825 5275
+F 0 "C3" H 1917 5321 50  0000 L CNN
+F 1 "0.1uF" H 1917 5230 50  0000 L CNN
+F 2 "Capacitor_SMD:C_0805_2012Metric" H 1825 5275 50  0001 C CNN
+F 3 "~" H 1825 5275 50  0001 C CNN
+	1    1825 5275
 	1    0    0    -1
 $EndComp
@@
 L Device:C_Small C4
 U 1 1 5C605212
-P 1975 5300
-F 0 "C4" H 2067 5346 50  0000 L CNN
-F 1 "0.1uF" H 2067 5255 50  0000 L CNN
-F 2 "Capacitor_SMD:C_0805_2012Metric" H 1975 5300 50  0001 C CNN
-F 3 "~" H 1975 5300 50  0001 C CNN
-	1    1975 5300
+P 2200 5275
+F 0 "C4" H 2292 5321 50  0000 L CNN
+F 1 "0.1uF" H 2292 5230 50  0000 L CNN
+F 2 "Capacitor_SMD:C_0805_2012Metric" H 2200 5275 50  0001 C CNN
+F 3 "~" H 2200 5275 50  0001 C CNN
+	1    2200 5275
 	1    0    0    -1
 $EndComp
@@
 L power:GND #PWR0105
 U 1 1 5C605AD7
-P 1525 5500
-F 0 "#PWR0105" H 1525 5250 50  0001 C CNN
-F 1 "GND" H 1530 5327 50  0000 C CNN
-F 2 "" H 1525 5500 50  0001 C CNN
-F 3 "" H 1525 5500 50  0001 C CNN
-	1    1525 5500
-	1    0    0    -1
-$EndComp
-Wire Wire Line
-	1525 5500 1525 5400
-Wire Wire Line
-	1525 5200 1525 5100
-Connection ~ 1675 5400
-Wire Wire Line
-	1975 5400 1675 5400
-Connection ~ 1675 5200
-Connection ~ 1375 5400
-Wire Wire Line
-	1075 5400 1375 5400
-Connection ~ 1375 5200
-Wire Wire Line
-	1375 5200 1075 5200
+P 1625 5475
+F 0 "#PWR0105" H 1625 5225 50  0001 C CNN
+F 1 "GND" H 1630 5302 50  0000 C CNN
+F 2 "" H 1625 5475 50  0001 C CNN
+F 3 "" H 1625 5475 50  0001 C CNN
+	1    1625 5475
+	1    0    0    -1
+$EndComp
+Wire Wire Line
+	1625 5475 1625 5375
 $Comp
 L power:+5V #PWR?
@@
 $EndComp
 $Comp
-L Switch:SW_Push SW?
-U 1 1 5C7BFB69
-P 1925 1475
-AR Path="/5C70FC4F/5C7BFB69" Ref="SW?"  Part="1"
-AR Path="/5C7BFB69" Ref="SW1"  Part="1"
-F 0 "SW1" H 1925 1760 50  0000 C CNN
-F 1 "SW_Push" H 1925 1669 50  0000 C CNN
-F 2 "Button_Switch_SMD:SW_SPST_SKQG_WithoutStem" H 1925 1675 50  0001 C CNN
-F 3 "" H 1925 1675 50  0001 C CNN
-	1    1925 1475
-	1    0    0    -1
-$EndComp
-$Comp
-L power:GND #PWR?
-U 1 1 5C7BFB71
-P 1625 1475
-AR Path="/5C70FC4F/5C7BFB71" Ref="#PWR?"  Part="1"
-AR Path="/5C7BFB71" Ref="#PWR0120"  Part="1"
-F 0 "#PWR0120" H 1625 1225 50  0001 C CNN
-F 1 "GND" H 1625 1325 50  0000 C CNN
-F 2 "" H 1625 1475 50  0001 C CNN
-F 3 "" H 1625 1475 50  0001 C CNN
-	1    1625 1475
-	1    0    0    -1
-$EndComp
-Wire Wire Line
-	1625 1475 1725 1475
-$Comp
 L power:GND #PWR0101
 U 1 1 5C7DAA6D
@@
 P 1300 1925
 AR Path="/5C70FC4F/5C83E985" Ref="SW?"  Part="1"
-AR Path="/5C83E985" Ref="SW2"  Part="1"
-F 0 "SW2" H 1300 1625 50  0000 C CNN
+AR Path="/5C83E985" Ref="SW1"  Part="1"
+F 0 "SW1" H 1300 1625 50  0000 C CNN
 F 1 "SW_SPDT" H 1300 1725 50  0000 C CNN
-F 2 "Button_Switch_SMD:SW_SPDT_PCM12" H 1300 1925 50  0001 C CNN
+F 2 "locallib:SW_SPDT_9.0x3.5mm" H 1300 1925 50  0001 C CNN
 F 3 "" H 1300 1925 50  0001 C CNN
 	1    1300 1925
@@
 L power:+3V3 #PWR0104
 U 1 1 5C9166F9
-P 1525 5100
-F 0 "#PWR0104" H 1525 4950 50  0001 C CNN
-F 1 "+3V3" H 1540 5273 50  0000 C CNN
-F 2 "" H 1525 5100 50  0001 C CNN
-F 3 "" H 1525 5100 50  0001 C CNN
-	1    1525 5100
+P 1625 5075
+F 0 "#PWR0104" H 1625 4925 50  0001 C CNN
+F 1 "+3V3" H 1640 5248 50  0000 C CNN
+F 2 "" H 1625 5075 50  0001 C CNN
+F 3 "" H 1625 5075 50  0001 C CNN
+	1    1625 5075
 	1    0    0    -1
 $EndComp
@@
 Wire Wire Line
 	5650 6700 5650 6600
-Connection ~ 5650 6600
 $Comp
 L Device:C_Small C9
@@
 $EndComp
 Wire Wire Line
-	7050 6600 7150 6600
-Wire Wire Line
-	7050 6700 7150 6700
-Wire Wire Line
 	7150 6700 7150 6600
-Connection ~ 7150 6600
 Wire Wire Line
 	7050 7000 7325 7000
@@
 Text GLabel 2125 1725 0    50   Input ~ 0
 PWRGD
-Wire Wire Line
-	2125 1725 2275 1725
-Wire Wire Line
-	2125 1475 2275 1475
-Wire Wire Line
-	2275 1475 2275 1725
-Connection ~ 2275 1725
-Wire Wire Line
-	2275 1725 2425 1725
 $Comp
 L Device:C_Small C5
 U 1 1 5D260E0E
-P 2250 5300
-F 0 "C5" H 2342 5346 50  0000 L CNN
-F 1 "4.7uF" H 2342 5255 50  0000 L CNN
-F 2 "Capacitor_SMD:C_0805_2012Metric" H 2250 5300 50  0001 C CNN
-F 3 "~" H 2250 5300 50  0001 C CNN
-	1    2250 5300
+P 2575 5275
+F 0 "C5" H 2667 5321 50  0000 L CNN
+F 1 "4.7uF" H 2667 5230 50  0000 L CNN
+F 2 "Capacitor_SMD:C_0805_2012Metric" H 2575 5275 50  0001 C CNN
+F 3 "~" H 2575 5275 50  0001 C CNN
+	1    2575 5275
 	1    0    0    -1
 $EndComp
@@
 L Device:C_Small C6
 U 1 1 5D2621C9
-P 2525 5300
-F 0 "C6" H 2617 5346 50  0000 L CNN
-F 1 "4.7uF" H 2617 5255 50  0000 L CNN
-F 2 "Capacitor_SMD:C_0805_2012Metric" H 2525 5300 50  0001 C CNN
-F 3 "~" H 2525 5300 50  0001 C CNN
-	1    2525 5300
-	1    0    0    -1
-$EndComp
-Wire Wire Line
-	1975 5200 2250 5200
-Connection ~ 1975 5200
-Connection ~ 2250 5200
-Wire Wire Line
-	2250 5200 2525 5200
-Connection ~ 1975 5400
-Connection ~ 2250 5400
-Wire Wire Line
-	2250 5400 1975 5400
+P 2950 5275
+F 0 "C6" H 3042 5321 50  0000 L CNN
+F 1 "4.7uF" H 3042 5230 50  0000 L CNN
+F 2 "Capacitor_SMD:C_0805_2012Metric" H 2950 5275 50  0001 C CNN
+F 3 "~" H 2950 5275 50  0001 C CNN
+	1    2950 5275
+	1    0    0    -1
+$EndComp
 $Comp
 L Device:C_Small C7
 U 1 1 5D29FD29
-P 2800 5300
-F 0 "C7" H 2892 5346 50  0000 L CNN
-F 1 "10nF" H 2892 5255 50  0000 L CNN
-F 2 "Capacitor_SMD:C_0805_2012Metric" H 2800 5300 50  0001 C CNN
-F 3 "~" H 2800 5300 50  0001 C CNN
-	1    2800 5300
+P 3325 5275
+F 0 "C7" H 3417 5321 50  0000 L CNN
+F 1 "10nF" H 3417 5230 50  0000 L CNN
+F 2 "Capacitor_SMD:C_0805_2012Metric" H 3325 5275 50  0001 C CNN
+F 3 "~" H 3325 5275 50  0001 C CNN
+	1    3325 5275
 	1    0    0    -1
 $EndComp
@@
 L Device:C_Small C8
 U 1 1 5D2A0066
-P 3075 5300
-F 0 "C8" H 3167 5346 50  0000 L CNN
-F 1 "1uF" H 3167 5255 50  0000 L CNN
-F 2 "Capacitor_SMD:C_0805_2012Metric" H 3075 5300 50  0001 C CNN
-F 3 "~" H 3075 5300 50  0001 C CNN
-	1    3075 5300
-	1    0    0    -1
-$EndComp
-Connection ~ 2525 5200
-Connection ~ 2525 5400
-Wire Wire Line
-	2525 5400 2250 5400
-Wire Wire Line
-	2525 5200 2800 5200
-Connection ~ 2800 5200
-Wire Wire Line
-	2800 5200 3075 5200
-Wire Wire Line
-	2525 5400 2800 5400
-Connection ~ 2800 5400
-Wire Wire Line
-	2800 5400 3075 5400
-Wire Wire Line
-	1375 5400 1525 5400
-Wire Wire Line
-	1525 5400 1675 5400
-Connection ~ 1525 5400
-Wire Wire Line
-	1675 5200 1975 5200
-Wire Wire Line
-	1525 5200 1375 5200
-Wire Wire Line
-	1675 5200 1525 5200
-Connection ~ 1525 5200
+P 3675 5275
+F 0 "C8" H 3767 5321 50  0000 L CNN
+F 1 "1uF" H 3767 5230 50  0000 L CNN
+F 2 "Capacitor_SMD:C_0805_2012Metric" H 3675 5275 50  0001 C CNN
+F 3 "~" H 3675 5275 50  0001 C CNN
+	1    3675 5275
+	1    0    0    -1
+$EndComp
 Text GLabel 4050 6575 2    50   Input ~ 0
 D-
@@
 Wire Wire Line
 	3325 1500 3500 1500
+Connection ~ 1450 5175
+Connection ~ 1450 5375
+Connection ~ 1825 5175
+Connection ~ 1825 5375
+Connection ~ 2200 5175
+Connection ~ 2200 5375
+Connection ~ 2575 5175
+Connection ~ 2575 5375
+Connection ~ 2950 5175
+Connection ~ 2950 5375
+Wire Wire Line
+	1825 5375 2200 5375
+Wire Wire Line
+	1075 5375 1450 5375
+Wire Wire Line
+	1075 5175 1450 5175
+Wire Wire Line
+	1825 5175 2200 5175
+Wire Wire Line
+	2575 5175 2950 5175
+Wire Wire Line
+	2575 5375 2950 5375
+Wire Wire Line
+	2200 5175 2575 5175
+Wire Wire Line
+	2950 5175 3325 5175
+Wire Wire Line
+	2200 5375 2575 5375
+Connection ~ 3325 5175
+Wire Wire Line
+	3325 5175 3675 5175
+Wire Wire Line
+	2950 5375 3325 5375
+Connection ~ 3325 5375
+Wire Wire Line
+	3325 5375 3675 5375
+Wire Wire Line
+	1625 5175 1625 5075
+Connection ~ 1625 5175
+Wire Wire Line
+	1625 5175 1825 5175
+Wire Wire Line
+	1450 5175 1625 5175
+Connection ~ 1625 5375
+Wire Wire Line
+	1625 5375 1825 5375
+Wire Wire Line
+	1450 5375 1625 5375
+Wire Wire Line
+	7150 6700 7050 6700
+Wire Wire Line
+	7050 6600 7150 6600
+Connection ~ 7150 6600
+Wire Wire Line
+	2125 1725 2425 1725
 $EndSCHEMATC

Commit message: rerouting of the USB and reg
Parts:
- K_#1, K_#10, K_#2, K_#3, K_#4, K_#5, K_#6, K_#7, K_#8, K_#9, K_'1, K_,1, K_-1, K_.1, K_/1, K_;1, K_=1, K_A1, K_ALT1, K_B1, K_BACK1, K_C1, K_CAPS1, K_CTRL1, K_D1, K_DELETE1, K_DOWN1, K_E1, K_ENTER1, K_ESC1, K_F1, K_FN1, K_G1, K_H1, K_I1, K_INSERT1, K_J1, K_K1, K_L1, K_LEFT1, K_M1, K_N1, K_O1, K_P1, K_Q1, K_R1, K_RALT1, K_RCTRL1, K_RIGHT1, K_RSHIFT1, K_S1, K_SHIFT1, K_SPACE1, K_T1, K_TAB1, K_U1, K_UP1, K_V1, K_W1, K_WIN1, K_X1, K_Y1, K_Z1, K_[1, K_]1: symbol MX_Alps_Hybrids:MX-1U -> board_arm-rescue:MX-1U-MX_Alps_Hybrids
- K_\1: symbol MX_Alps_Hybrids:MX-1.5U -> board_arm-rescue:MX-1.5U-MX_Alps_Hybrids
- USB1: symbol Type-C:HRO-TYPE-C-31-M-12 -> board_arm-rescue:HRO-TYPE-C-31-M-12-Type-C
Connections:
- net COL0: no longer K_CAPS1.1 (COL), K_ESC1.1 (COL), K_SHIFT1.1 (COL), K_TAB1.1 (COL)
- net COL1: no longer K_#1.1 (COL), K_A1.1 (COL), K_Q1.1 (COL)
- net COL10: no longer K_#10.1 (COL), K_.1.1 (COL), K_;1.1 (COL), K_P1.1 (COL)
- net COL11: no longer K_'1.1 (COL), K_-1.1 (COL), K_/1.1 (COL), K_[1.1 (COL)
- net COL12: no longer K_=1.1 (COL), K_RSHIFT1.1 (COL), K_]1.1 (COL)
- net COL13: no longer K_BACK1.1 (COL), K_ENTER1.1 (COL), K_\1.1 (COL)
- net COL14: no longer K_UP1.1 (COL)
- net COL15: no longer K_DELETE1.1 (COL), K_INSERT1.1 (COL)
- net COL2: no longer K_#2.1 (COL), K_S1.1 (COL), K_W1.1 (COL), K_Z1.1 (COL)
- net COL3: no longer K_#3.1 (COL), K_D1.1 (COL), K_E1.1 (COL)
- net COL4: no longer K_#4.1 (COL), K_F1.1 (COL), K_R1.1 (COL)
- net COL5: no longer K_#5.1 (COL), K_G1.1 (COL), K_T1.1 (COL)
- net COL6: no longer K_#6.1 (COL), K_B1.1 (COL), K_H1.1 (COL), K_Y1.1 (COL)
- net COL7: no longer K_#7.1 (COL), K_J1.1 (COL), K_U1.1 (COL)
- net COL8: no longer K_#8.1 (COL), K_I1.1 (COL), K_K1.1 (COL)
- net COL9: no longer K_#9.1 (COL), K_L1.1 (COL), K_O1.1 (COL)
