File: board_arm.sch (KiCad schematic (older format))
At the start: 155 parts, among them SW1 SW_SPDT, U1 STM32F072CBT6, U2 PRTR5V0U2X, U3 MCP1725-3302E_SN

Commit message: Ajout de TP GND, 3V3 et reset pour SWD
Parts:
- added 3V3, GND1, RESET1: TestPoint, TestPoint:TestPoint_Pad_D1.0mm, symbol Connector:TestPoint
- renumbered TP2 to SWCLK1, TP1 to SWDIO1
Connections:
- net +3V3: now also 3V3.1
- net GND: now also GND1.1
- net PWRGD: now also RESET1.1
Changed lines of the file:
@@
 	9175 2050 9175 2175
 $Comp
-L Connector:TestPoint TP1
+L Connector:TestPoint SWDIO1
 U 1 1 5C6EFC1B
 P 8900 6800
-F 0 "TP1" H 8958 6920 50  0000 L CNN
+F 0 "SWDIO1" H 8958 6920 50  0000 L CNN
 F 1 "TestPoint" H 8958 6829 50  0000 L CNN
 F 2 "TestPoint:TestPoint_Pad_D1.0mm" H 9100 6800 50  0001 C CNN
@@
 SWDCLK
 $Comp
-L Connector:TestPoint TP2
+L Connector:TestPoint SWCLK1
 U 1 1 5C7259A1
 P 9500 6800
-F 0 "TP2" H 9558 6920 50  0000 L CNN
+F 0 "SWCLK1" H 9558 6920 50  0000 L CNN
 F 1 "TestPoint" H 9558 6829 50  0000 L CNN
 F 2 "TestPoint:TestPoint_Pad_D1.0mm" H 9700 6800 50  0001 C CNN
@@
 $EndComp
 $Comp
-L power:GND #PWR?
+L power:GND #PWR0117
 U 1 1 5C976169
 P 4275 3800
-F 0 "#PWR?" H 4275 3550 50  0001 C CNN
+F 0 "#PWR0117" H 4275 3550 50  0001 C CNN
 F 1 "GND" H 4280 3627 50  0000 C CNN
 F 2 "" H 4275 3800 50  0001 C CNN
@@
 Wire Wire Line
 	4275 3625 4225 3625
+Text GLabel 10050 6800 3    50   Input ~ 0
+PWRGD
+$Comp
+L Connector:TestPoint RESET1
+U 1 1 5C89FE58
+P 10050 6800
+F 0 "RESET1" H 10108 6920 50  0000 L CNN
+F 1 "TestPoint" H 10108 6829 50  0000 L CNN
+F 2 "TestPoint:TestPoint_Pad_D1.0mm" H 10250 6800 50  0001 C CNN
+F 3 "~" H 10250 6800 50  0001 C CNN
+	1    10050 6800
+	1    0    0    -1
+$EndComp
+$Comp
+L Connector:TestPoint 3V3
+U 1 1 5C8D840B
+P 9225 7625
+F 0 "3V3" H 9283 7745 50  0000 L CNN
+F 1 "TestPoint" H 9283 7654 50  0000 L CNN
+F 2 "TestPoint:TestPoint_Pad_D1.0mm" H 9425 7625 50  0001 C CNN
+F 3 "~" H 9425 7625 50  0001 C CNN
+	1    9225 7625
+	-1   0    0    1
+$EndComp
+$Comp
+L Connector:TestPoint GND1
+U 1 1 5C8F4376
+P 9775 7675
+F 0 "GND1" H 9833 7795 50  0000 L CNN
+F 1 "TestPoint" H 9833 7704 50  0000 L CNN
+F 2 "TestPoint:TestPoint_Pad_D1.0mm" H 9975 7675 50  0001 C CNN
+F 3 "~" H 9975 7675 50  0001 C CNN
+	1    9775 7675
+	1    0    0    -1
+$EndComp
+$Comp
+L power:+3V3 #PWR0118
+U 1 1 5C99C6DC
+P 9225 7625
+F 0 "#PWR0118" H 9225 7475 50  0001 C CNN
+F 1 "+3V3" H 9240 7798 50  0000 C CNN
+F 2 "" H 9225 7625 50  0001 C CNN
+F 3 "" H 9225 7625 50  0001 C CNN
+	1    9225 7625
+	1    0    0    -1
+$EndComp
+$Comp
+L power:GND #PWR0119
+U 1 1 5C9F054E
+P 9775 7675
+F 0 "#PWR0119" H 9775 7425 50  0001 C CNN
+F 1 "GND" H 9780 7502 50  0000 C CNN
+F 2 "" H 9775 7675 50  0001 C CNN
+F 3 "" H 9775 7675 50  0001 C CNN
+	1    9775 7675
+	1    0    0    -1
+$EndComp
 $EndSCHEMATC
